File: PCB/Twin_PLL_GPSDO.brd (EAGLE design)
At the start: 109 x 63 mm, 107 parts, among them IC6 7805DT, IC7 7809DT, IC8 LD1117AS33TR, U1 RASPBERRY_PICOTH, U2 ADF4351BCPZ, U3 ADF4351BCPZ

Commit message: PCB catchup
Parts:
- removed C28: 1nF, resistor:C0603
- removed IC8: LD1117AS33TR, v-reg:SOT223
- added C70, C71: 100nF, rcl:C0805
- added IC1, IC2: ADP151WAUJZ-1.8-R7, ADP151WAUJZ-1.8-R7:SOT95P280X100-5N
- added IC3: MCP4725A0T-E_CH, MCP4725A0T-E_CH:SOT95P270X145-6N
- added R11: 1K0, resistor:R0805
- added R12, R13: 100R, resistor:R0805
- added U$2: GPS, gps:GPS
- C38: value 100pF -> 100nF; device resistor:C0603 -> rcl:C0603
- moved C38 78.8 mm to (24.0, 23.3)
- moved C30 53.5 mm to (69.5, 17.5)
- moved C31 52.6 mm to (69.5, 15.5)
- moved C24 28.6 mm to (28.4, 20.4)
- moved C25 28.5 mm to (30.4, 20.4)
- moved U1 27.3 mm to (27.0, 40.3)
- moved C29 24.2 mm to (44.3, 5.40), turned to 90 degrees
- moved OSC1 22.6 mm to (40.1, 14.7)
- moved SCK3 22.2 mm to (0.64, 7.78)
- moved SCK4 21.0 mm to (0.64, 23.0)
- moved SCK2 2.83 mm to (107.8, 38.4)
- moved SCK1 1.41 mm to (108.0, 14.0)
Connections:
- removed net 10_MHZ_4001: C28.1
- removed net LO1_CE: R2.1, R4.1, U2.4, U3.4
- removed net LO1_LE: U2.3
- removed net LO1_LOCK_DETECT: U2.25
- removed net LO2_LE: U3.3
- removed net LO2_LOCK_DETECT: U3.25
- removed net LO_MOSI: U2.2, U3.2
- removed net LO_SCK: U2.1, U3.1
- new net +3V3_ADF1: C1.2, C27.1, C48.2, C49.2, C50.2, C51.2, C69.2, IC1.5, L27.2, L30.1, L31.2, L32.1, R2.2, R38.2, R39.2, U2.10, U2.26
- new net +3V3_ADF2: C32.2, C34.2, C60.2, C61.2, C62.2, C63.2, C71.1, IC2.5, L1.1, L2.1, L3.2, L4.2, R10.2, R4.2, R9.2, U3.10, U3.26
- new net 1PPS: U1.4
- new net 1_PPS: U$2.P$1
- new net 3V3: U$2.P$5
- new net ADF1_CE: R2.1, U1.16, U2.4
- new net ADF1_CLK: U1.9, U2.1
- new net ADF1_LD: U1.14, U2.25
- new net ADF1_LE: U1.6, U2.3
- new net ADF1_MOSI: U1.7, U2.2
- new net ADF2_CE: R4.1, U1.17, U3.4
- new net ADF2_CLK: U1.10, U3.1
- new net ADF2_LD: U1.15, U3.25
- new net ADF2_LE: U1.12, U3.3
- new net ADF2_MOSI: U1.11, U3.2
- new net ALARM_PIN: U1.27
- new net DEBUG_TX_PIN: U1.29
- new net FREQ_COUNT_IN: R12.1, U1.5
- new net GPS_RX: U$2.P$2, U1.2
- new net GPS_TX: U$2.P$3, U1.1
- new net I2C_SCL: IC3.5, U1.20
- new net I2C_SDA: IC3.4, U1.19
- new net LED_ADF1_LOCK: U1.24
- new net LED_ADF2_LOCK: U1.25
- new net LED_ALARM: U1.26
- new net LED_GPS_DISC: U1.22
- new net LED_GPS_LOCK: U1.21
- new net LED_SATS_BLINK: U1.31
- new net LED_SATS_USED: U1.32
- new net N$26: C29.1, R13.2
- new net N$27: C29.2
- net +3V3: now also C38.1, IC3.2; no longer C1.2, C27.1, C32.2, C34.2, C48.2, C49.2, C50.2, C51.2, C60.2, C61.2, C62.2, C63.2, C69.2, IC8.4, L1.1, L2.1, L27.2, L3.2, L30.1, L31.2, L32.1, L4.2, R10.2, R2.2, R38.2, R39.2, R4.2, R9.2, U2.10, U2.26, U3.10, U3.26
- net +5V: now also C26.1, C70.1, IC1.1, IC1.3, IC2.1, IC2.3
- net +9V: no longer C26.1, IC8.3
- net 10MHZ: now also R12.2, R13.1; no longer C28.2, C29.1
- net GND: now also C36.2, C37.2, C38.2, C70.2, C71.2, IC1.2, IC2.2, IC3.3, IC3.6, U$2.P$4; no longer IC8.1
- net N$101: now also SCK1.1
- net N$20: now also IC3.1, R11.1; no longer C65.2
- net N$32: now also R11.2
- net OUTPUT: now also C65.2; no longer C38.2
Routing:
- net 10MHZ_REF: track 1060.1 -> 3.80 mm
- net LO_SCK: track 644.9 -> 0.00 mm, vias 2 -> 0
- net N$16: track 638.2 -> 3.81 mm
- net LO_MOSI: track 547.7 -> 0.00 mm, vias 2 -> 0
- net N$50: track 387.4 -> 3.81 mm
- net ADF1_LE: track 0.00 -> 105.0 mm, vias 0 -> 1
- net ADF1_MOSI: track 0.00 -> 99.0 mm, vias 0 -> 1
- net ADF1_CLK: track 0.00 -> 92.2 mm, vias 0 -> 1
- net GPS_TX: track 0.00 -> 62.0 mm
- net +3V3_ADF1: track 0.00 -> 60.1 mm, vias 0 -> 4
- net +3V3_ADF2: track 0.00 -> 56.0 mm, vias 0 -> 4
- net GPS_RX: track 0.00 -> 55.7 mm, vias 0 -> 2
- net FREQ_COUNT_IN: track 0.00 -> 54.7 mm, vias 0 -> 1
- net +3V3: track 52.7 -> 3.34 mm, vias 4 -> 0
- net ADF1_CE: track 0.00 -> 20.5 mm
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- removed copper zone on layer 15, net GND
