File: PCB/Twin_PLL_GPSDO.brd (EAGLE design)
At the start: 109 x 63 mm, 114 parts, among them IC1 ADP151WAUJZ-1.8-R7, IC2 ADP151WAUJZ-1.8-R7, IC3 MCP4725A0T-E_CH, IC6 7805DT, IC7 7809DT, U1 RASPBERRY_PICOTH, U2 ADF4351BCPZ, U3 ADF4351BCPZ

Commit message: JLC Build, v 1.1
Parts:
- removed IC6: 7805DT, linear:TO252
- removed IC7: 7809DT, linear:TO252
- removed LSP1, LSP2: LSP13, solpad:LSP13
- removed SCK3, SCK4: SMA-142-0701-871/876, con-coax:J502-ND-142-0701-871/876
- added C28, C72: 22uF, resistor:C1210
- added C73: 100nF, rcl:C0805
- added C74: 10uF, rcl:C0805
- added IC4: LT1963AEQ-2.5#PBF, LT1963AEQ-2.5#PBF:LT1963AEQ25PBF
- added L5: DFE322512F-3R3M=P2, DFE322512F-3R3M=P2:1277ASH100MP2
- added L6, L7, L9: 100nH, resistor:R0603
- added LED1, LED2, LED3, LED4: (no value), led:CHIPLED_0603
- added PS1: LMR33630ADDA, LMR33630ADDA:SOIC127P600X170-9N
- added R14, R15, R16, R17: 1K0, resistor:R0805
- added R18, R19, R20, R21, R22: 330R, resistor:R0603
- added R23: 1k, resistor:R0603
- added R24: 330R, resistor:R0805
- added R25: 10K, rcl:R0805
- added R26: 4k7, resistor:R0603
- added T1: BC847, transistor:SOT23
- added TR4: SI2309, transistor-small-signal:SOT23
- C11, C13, C15, C3, C34, C35, C4, C41, C44, C47, C50, C57, C59, C62, C69, C7, C9: value 100N -> 100nF
- C18: value 10uF -> 22uF; device rcl:C0805 -> resistor:C1210
- C21: value 100nF -> 1uF
- C29: value 1nF -> 100nF; device resistor:C0603 -> rcl:C0805
- C52, C64: value 100pF -> 1nF; device rcl:C0603 -> resistor:C0603
- L1, L2, L27, L3, L30, L31, L32, L4: value (none) -> 100nH
- R13: value 100R -> 3k3; device resistor:R0805 -> resistor:R0603
- U1: value RASPBERRY_PICOTH -> (none); device RpiPico:PICO-PKG-TH -> RpiPico:PICO-PKG-TH-STD
- moved L8 134.7 mm to (58.8, 14.2), turned to 90 degrees
- moved C37 130.8 mm to (60.9, 14.2), turned to 90 degrees
- moved C21 130.4 mm to (9.21, 10.8), turned to 270 degrees
- moved C36 130.2 mm to (63.2, 14.2), turned to 90 degrees
- moved C20 121.4 mm to (10.2, 25.1), turned to 0 degrees
- moved C18 114.1 mm to (24.4, 7.94)
- moved C19 114.0 mm to (10.2, 22.9), turned to 0 degrees
- moved C16 100.8 mm to (44.5, 20.0), turned to 90 degrees
- moved C22 99.8 mm to (11.4, 10.8)
- moved C23 99.7 mm to (41.8, 21.0), turned to 90 degrees
- moved C27 94.9 mm to (75.0, 18.2)
- moved C17 91.7 mm to (46.7, 19.4), turned to 90 degrees
- moved C26 69.0 mm to (72.4, 39.6), turned to 90 degrees
- moved R12 56.1 mm to (78.4, 23.8), turned to 180 degrees
- moved C25 40.1 mm to (68.2, 7.03)
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Connections:
- removed net +3V3: C38.1, IC3.2, L8.2
- removed net +9V: C20.1, C21.1, C22.1, IC7.2
- removed net 1PPS: U1.4
- removed net 3V3: U$2.P$5
- removed net ADF1_CLK: U1.9, U2.1
- removed net ADF1_MOSI: U1.7, U2.2
- removed net ADF2_CLK: U1.10, U3.1
- removed net ADF2_MOSI: U1.11, U3.2
- removed net DEBUG_TX_PIN: U1.29
- removed net LED_ALARM: U1.26
- removed net LED_SATS_BLINK: U1.31
- removed net LED_SATS_USED: U1.32
- removed net SWGND: U1.42
- removed net VSYS: U1.39
- new net ADF_CLK: U1.9, U2.1, U3.1
- new net ADF_MOSI: U1.11, U2.2, U3.2
- new net ALARM_OUT: R24.1
- new net N$29: IC4.5, R15.2, R16.1
- new net N$31: PS1.5, R14.1, R17.2
- new net N$33: C21.1, PS1.6
- new net N$34: C22.1, PS1.7
- new net N$35: C22.2, L5.1, PS1.8
- new net N$36: C17.1, C18.1, C28.1, C72.1, IC4.1, IC4.2, L5.2, R14.2
- new net N$37: LED2.A, R19.1
- new net N$38: LED3.A, R20.1
- new net N$39: LED4.A, R21.1
- new net N$41: C64.1, L6.2, L7.1
- new net N$42: R25.1, TR4.1
- new net N$43: C52.1, L7.2, L9.1
- new net SWITCH: R24.2, TR4.3
- net +12V: now also C20.1, PS1.2, PS1.3; no longer IC7.1, LSP1.MP
- net +12V_OSC: no longer IC6.1, LSP2.MP
- net +5V: now also C29.1, C73.1, C74.1, IC4.4, L8.2, R15.1, R23.1, TR4.2, U$2.P$5, U1.39; no longer C17.1, C18.1, IC6.2
- net 10MHZ_REF: now also L9.2
- net 1_PPS: now also U1.34
- net ALARM_PIN: now also R22.1, U1.1; no longer U1.27
- net AVDD: now also C38.1, IC3.2
- net FREQ_COUNT_IN: now also U1.29; no longer U1.5
- net GND: now also C28.2, C29.2, C52.2, C64.2, C72.2, C73.2, C74.2, IC4.3, IC4.6, LED1.C, LED2.C, LED3.C, LED4.C, PS1.1, PS1.9, R16.2, R17.1, R26.1, T1.2; no longer C22.2, IC6.3, IC7.3, SCK3.G@1, SCK3.G@2, SCK3.G@3, SCK3.G@4, SCK4.G@1, SCK4.G@2, SCK4.G@3, SCK4.G@4
- net GPS_RX: now also U1.26; no longer U1.2
- net GPS_TX: now also U1.27; no longer U1.1
- net LED_ADF1_LOCK: now also R19.2
- net LED_ADF2_LOCK: now also R20.2
- net LED_GPS_DISC: now also R18.2, U1.21; no longer U1.22
- net LED_GPS_LOCK: now also R21.2, U1.22; no longer U1.21
- net N$18: no longer C52.1
- net N$21: now also R23.2, R25.2, T1.3; no longer C64.2
- net N$26: now also L6.1, R26.2; no longer C29.1
- net N$27: now also LED1.A, R18.1; no longer C29.2
- net N$28: now also R22.2, T1.1; no longer C52.2
- net N$7: no longer C64.1
Routing:
- net +5V: track 14.3 -> 199.1 mm, vias 0 -> 4
- net ADF_CLK: track 0.00 -> 110.4 mm, vias 0 -> 4
- net ADF_MOSI: track 0.00 -> 108.7 mm, vias 0 -> 2
- net ADF1_MOSI: track 99.0 -> 0.00 mm, vias 1 -> 0
- net GND: track 92.7 -> 189.7 mm, vias 123 -> 137
- net ADF1_CLK: track 92.2 -> 0.00 mm, vias 1 -> 0
- net ADF2_LE: track 0.00 -> 72.0 mm, vias 0 -> 1
- net ADF2_CE: track 3.17 -> 67.4 mm, vias 0 -> 3
- net ADF1_CE: track 20.5 -> 83.3 mm, vias 0 -> 3
- net N$36: track 0.00 -> 61.9 mm, vias 0 -> 2
- net ADF1_LD: track 19.9 -> 78.3 mm, vias 2 -> 5
- net ADF2_LD: track 0.00 -> 54.9 mm, vias 0 -> 1
- net I2C_SDA: track 0.00 -> 51.0 mm
- net I2C_SCL: track 0.00 -> 46.2 mm
- net GPS_TX: track 62.0 -> 17.5 mm
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- added copper zone on layer 16, net +12V
- added copper zone on layer 16, net ALARM_OUT
Other:
- board text added: "G1YFG"
- board text added: "GPS"
- board text added: "LOCK"
- board text added: "PLL1"
- board text added: "PLL2"
- board text added: "V 1.1"
- board text removed: ">PLOT_DATE_TIME"
- board text removed: "EXT LOCK"
- board text removed: "EXT REF"
- board text removed: "G1YFG Microwave Local Oscillator"
- board text removed: "VCO LOCK"
