File: PCB/Twin_PLL_GPSDO.brd (EAGLE design)
At the start: 109 x 63 mm, 136 parts, among them IC1 ADP151WAUJZ-1.8-R7, IC2 ADP151WAUJZ-1.8-R7, IC3 MCP4725A0T-E_CH, IC4 LT1963AEQ-2.5#PBF, T1 BC847, U2 ADF4351BCPZ, U3 ADF4351BCPZ

Commit message: Ketchup
Parts:
- added D1, D2: (no value), diode:SOD123
- added R27, R28: 10K, resistor:R0603
- moved C38 1.63 mm to (60.8, 11.3), turned to 180 degrees
Connections:
- new net N$40: D1.C, U1.39
- new net N$44: D2.A, R24.1
- net +5V: now also D1.A, R27.2, R28.2; no longer U1.39
- net ALARM_OUT: now also D2.C; no longer R24.1
- net AVDD: now also C38.2, IC3.3; no longer C38.1, IC3.2
- net GND: now also C38.1, IC3.2; no longer C38.2, IC3.3
- net I2C_SCL: now also R27.1
- net I2C_SDA: now also R28.1
Routing:
- net +5V: track 199.1 -> 241.7 mm, vias 4 -> 5
- net ALARM_OUT: track 34.5 -> 0.00 mm, vias 2 -> 0
- net N$40: track 0.00 -> 8.97 mm
- net I2C_SCL: track 46.1 -> 48.8 mm
- net I2C_SDA: track 51.8 -> 54.4 mm
- net AVDD: track 11.1 -> 10.1 mm

Commit message: initial corrections to producion PCB
Parts:
- removed R36, R7: 0R, rcl:R0603
- removed R37, R8: NF, rcl:R0603
- moved D2 67.2 mm to (28.9, 38.7)
- moved C19 4.55 mm to (14.3, 24.8), turned to 90 degrees
- moved C28 3.51 mm to (24.4, 8.26)
- moved PS1 3.51 mm to (13.3, 17.8)
- moved C18 3.51 mm to (27.9, 8.26)
- moved C21 3.51 mm to (12.7, 11.1)
- moved C22 3.51 mm to (14.9, 11.1)
- moved C72 3.51 mm to (21.0, 8.26)
- moved R14 3.51 mm to (12.7, 6.67)
- moved R17 3.51 mm to (10.5, 6.67)
- moved C20 1.93 mm to (12.1, 24.8), turned to 90 degrees
- moved L5 1.00 mm to (21.0, 13.3), turned to 270 degrees
- moved L27 0.08 mm to (98.3, 19.2)
Connections:
- removed net N$15: R5.2, R7.2, R8.1
- removed net N$16: R8.2, U3.5
- removed net N$49: R34.2, R36.2, R37.1
- removed net N$50: R37.2, U2.5
- net GND: now also R34.2, R5.2; no longer R36.1, R7.1
Routing:
- net ALARM_OUT: track 0.00 -> 49.3 mm, vias 0 -> 3
- net N$16: track 23.6 -> 0.00 mm, vias 2 -> 0
- net N$50: track 22.9 -> 0.00 mm, vias 2 -> 0
- net N$44: track 0.00 -> 8.57 mm
- net GND: track 170.9 -> 167.4 mm
- net N$49: track 3.35 -> 0.00 mm
- net N$15: track 3.35 -> 0.00 mm
- net +12V: track 8.35 -> 11.2 mm
- net N$35: track 13.1 -> 12.2 mm
