File: PCB/Twin_PLL_GPSDO.sch (EAGLE design)
At the start: 107 parts, among them IC6 7805DT, IC7 7809DT, IC8 LD1117AS33TR, U1 RASPBERRY_PICOTH, U2 ADF4351BCPZ, U3 ADF4351BCPZ

Commit message: PCB catchup
Parts:
- removed C28: 1nF, resistor:C-EUC0603
- removed IC8: LD1117AS33TR, v-reg:LD117ASTR
- added C70, C71: 100nF, rcl:C-EUC0805
- added IC1, IC2: ADP151WAUJZ-1.8-R7, ADP151WAUJZ-1.8-R7:ADP151WAUJZ-1.8-R7
- added IC3: MCP4725A0T-E_CH, MCP4725A0T-E_CH:MCP4725A0T-E_CH
- added R11: 1K0, resistor:R-EU_R0805
- added R12, R13: 100R, resistor:R-EU_R0805
- added U$2: GPS, gps:GPS
- C38: value 100pF -> 100nF; device resistor:C-EUC0603 -> rcl:C-EUC0603
Connections:
- removed net 10_MHZ_4001: C28.1
- removed net LO1_CE: R2.1, R4.1, U2G$1.CE, U3G$1.CE
- removed net LO1_LE: U2G$1.LE
- removed net LO1_LOCK_DETECT: U2G$1.LD
- removed net LO2_LE: U3G$1.LE
- removed net LO2_LOCK_DETECT: U3G$1.LD
- removed net LO_MOSI: U2G$1.DATA, U3G$1.DATA
- removed net LO_SCK: U2G$1.CLK, U3G$1.CLK
- new net +3V3_ADF1: C1.2, C27.1, C48.2, C49.2, C50.2, C51.2, C69.2, IC1.VOUT, L27.2, L30.1, L31.2, L32.1, R2.2, R38.2, R39.2, U2G$1.AVDD, U2G$1.PDBRF
- new net +3V3_ADF2: C32.2, C34.2, C60.2, C61.2, C62.2, C63.2, C71.1, IC2.VOUT, L1.1, L2.1, L3.2, L4.2, R10.2, R4.2, R9.2, U3G$1.AVDD, U3G$1.PDBRF
- new net 1PPS: U1.GP2
- new net 1_PPS: U$2.1_PPS
- new net 3V3: U$2.VCC
- new net ADF1_CE: R2.1, U1.GP12, U2G$1.CE
- new net ADF1_CLK: U1.GP4, U2G$1.CLK
- new net ADF1_LD: U1.GP10, U2G$1.LD
- new net ADF1_LE: U1.GP6, U2G$1.LE
- new net ADF1_MOSI: U1.GP5, U2G$1.DATA
- new net ADF2_CE: R4.1, U1.GP13, U3G$1.CE
- new net ADF2_CLK: U1.GP7, U3G$1.CLK
- new net ADF2_LD: U1.GP11, U3G$1.LD
- new net ADF2_LE: U1.GP9, U3G$1.LE
- new net ADF2_MOSI: U1.GP8, U3G$1.DATA
- new net ALARM_PIN: U1.GP21
- new net DEBUG_TX_PIN: U1.GP22
- new net FREQ_COUNT_IN: R12.1, U1.GP3
- new net GPS_RX: U$2.TXD, U1.GP1
- new net GPS_TX: U$2.RXD, U1.GP0
- new net I2C_SCL: IC3.SCL, U1.GP15
- new net I2C_SDA: IC3.SDA, U1.GP14
- new net LED_ADF1_LOCK: U1.GP18
- new net LED_ADF2_LOCK: U1.GP19
- new net LED_ALARM: U1.GP20
- new net LED_GPS_DISC: U1.GP17
- new net LED_GPS_LOCK: U1.GP16
- new net LED_SATS_BLINK: U1.GP26
- new net LED_SATS_USED: U1.GP27
- new net N$26: C29.1, R13.2
- new net N$27: C29.2
- net +3V3: now also C38.1, IC3.VSS; no longer C1.2, C27.1, C32.2, C34.2, C48.2, C49.2, C50.2, C51.2, C60.2, C61.2, C62.2, C63.2, C69.2, IC8.OUT, L1.1, L2.1, L27.2, L3.2, L30.1, L31.2, L32.1, L4.2, R10.2, R2.2, R38.2, R39.2, R4.2, R9.2, U2G$1.AVDD, U2G$1.PDBRF, U3G$1.AVDD, U3G$1.PDBRF
- net +5V: now also C26.1, C70.1, IC1.EN, IC1.VIN, IC2.EN, IC2.VIN
- net +9V: no longer C26.1, IC8.IN
- net 10MHZ: now also R12.2, R13.1; no longer C28.2, C29.1
- net GND: now also C36.2, C37.2, C38.2, C70.2, C71.2, IC1.GND, IC2.GND, IC3.A0, IC3.VDD, SCK1G1.GND, U$2.GND; no longer IC8.ADJ
- net N$101: now also SCK1G1.1
- net N$20: now also IC3.VOUT, R11.1; no longer C65.2
- net N$32: now also R11.2
- net OUTPUT: now also C65.2; no longer C38.2
