File: PCB/Twin_PLL_GPSDO.sch (EAGLE design)
At the start: 114 parts, among them IC1 ADP151WAUJZ-1.8-R7, IC2 ADP151WAUJZ-1.8-R7, IC3 MCP4725A0T-E_CH, IC6 7805DT, IC7 7809DT, U1 RASPBERRY_PICOTH, U2 ADF4351BCPZ, U3 ADF4351BCPZ

Commit message: JLC Build, v 1.1
Parts:
- removed IC6: 7805DT, linear:7805DT
- removed IC7: 7809DT, linear:7805DT
- removed LSP1, LSP2: LSP13, solpad:LSP13
- removed SCK3, SCK4: SMA-142-0701-871/876, con-coax:SMA-142-0701-871/876
- added C28, C72: 22uF, resistor:C-EUC1210
- added C73: 100nF, rcl:C-EUC0805
- added C74: 10uF, rcl:C-EUC0805
- added IC4: LT1963AEQ-2.5#PBF, LT1963AEQ-2.5#PBF:LT1963AEQ-2.5#PBF
- added L5: DFE322512F-3R3M=P2, DFE322512F-3R3M=P2:DFE322512F-3R3M=P2
- added L6, L7, L9: 100nH, resistor:R-EU_R0603
- added LED1, LED2, LED3, LED4: (no value), led:LEDCHIPLED_0603
- added PS1: LMR33630ADDA, LMR33630ADDA:LMR33630ADDA
- added R14, R15, R16, R17: 1K0, resistor:R-EU_R0805
- added R18, R19, R20, R21, R22: 330R, resistor:R-EU_R0603
- added R23: 1k, resistor:R-EU_R0603
- added R24: 330R, resistor:R-EU_R0805
- added R25: 10K, rcl:R-EU_R0805
- added R26: 4k7, resistor:R-EU_R0603
- added T1: BC847, transistor:BC847
- added TR4: SI2309, transistor-small-signal:BSS84
- C11, C13, C15, C3, C34, C35, C4, C41, C44, C47, C50, C57, C59, C62, C69, C7, C9: value 100N -> 100nF
- C18: value 10uF -> 22uF; device rcl:C-EUC0805 -> resistor:C-EUC1210
- C21: value 100nF -> 1uF
- C29: value 1nF -> 100nF; device resistor:C-EUC0603 -> rcl:C-EUC0805
- C52, C64: value 100pF -> 1nF; device rcl:C-EUC0603 -> resistor:C-EUC0603
- L1, L2, L27, L3, L30, L31, L32, L4: value (none) -> 100nH
- R13: value 100R -> 3k3; device resistor:R-EU_R0805 -> resistor:R-EU_R0603
- U1: value RASPBERRY_PICOTH -> (none); device RpiPico:RASPBERRY_PICOTH -> RpiPico:RASPBERRY_PICO-NO_DEBUGTH
Connections:
- removed net +3V3: C38.1, IC3.VSS, L8.2
- removed net +9V: C20.1, C21.1, C22.1, IC7.VO
- removed net 1PPS: U1.GP2
- removed net 3V3: U$2.VCC
- removed net ADF1_CLK: U1.GP4, U2G$1.CLK
- removed net ADF1_MOSI: U1.GP5, U2G$1.DATA
- removed net ADF2_CLK: U1.GP7, U3G$1.CLK
- removed net ADF2_MOSI: U1.GP8, U3G$1.DATA
- removed net DEBUG_TX_PIN: U1.GP22
- removed net LED_ALARM: U1.GP20
- removed net LED_SATS_BLINK: U1.GP26
- removed net LED_SATS_USED: U1.GP27
- new net ADF_CLK: U1.GP6, U2G$1.CLK, U3G$1.CLK
- new net ADF_MOSI: U1.GP8, U2G$1.DATA, U3G$1.DATA
- new net ALARM_OUT: R24.1
- new net N$29: IC4.SENSE, R15.2, R16.1
- new net N$31: PS1.FB, R14.1, R17.2
- new net N$33: C21.1, PS1.VCC
- new net N$34: C22.1, PS1.BOOT
- new net N$35: C22.2, L5.1, PS1.SW
- new net N$36: C17.1, C18.1, C28.1, C72.1, IC4.!SHDN, IC4.IN, L5.2, R14.2
- new net N$37: LED2.A, R19.1
- new net N$38: LED3.A, R20.1
- new net N$39: LED4.A, R21.1
- new net N$41: C64.1, L6.2, L7.1
- new net N$42: R25.1, TR4.G
- new net N$43: C52.1, L7.2, L9.1
- new net SWITCH: R24.2, TR4.D
- net +12V: now also C20.1, PS1.EN, PS1.VIN; no longer IC7.VI, LSP1.MP
- net +12V_OSC: no longer IC6.VI, LSP2.MP
- net +5V: now also C29.1, C73.1, C74.1, IC4.OUT, L8.2, R15.1, R23.1, TR4.S, U$2.VCC, U1.VSYS; no longer C17.1, C18.1, IC6.VO
- net 10MHZ_REF: now also L9.2
- net 1_PPS: now also U1.GP28
- net ADF1_LE: now also U1.GP4; no longer U1.GP6
- net ALARM_PIN: now also R22.1, U1.GP0; no longer U1.GP21
- net AVDD: now also C38.1, IC3.VSS
- net FREQ_COUNT_IN: now also U1.GP22; no longer U1.GP3
- net GND: now also C28.2, C29.2, C52.2, C64.2, C72.2, C73.2, C74.2, IC4.GND_1, IC4.GND_2, LED1.C, LED2.C, LED3.C, LED4.C, PS1.EP, PS1.PGND, R16.2, R17.1, R26.1, T1.E, U1.GND; no longer C22.2, IC6.GND, IC7.GND
- net GPS_RX: now also U1.GP20; no longer U1.GP1
- net GPS_TX: now also U1.GP21; no longer U1.GP0
- net LED_ADF1_LOCK: now also R19.2
- net LED_ADF2_LOCK: now also R20.2
- net LED_GPS_DISC: now also R18.2, U1.GP16; no longer U1.GP17
- net LED_GPS_LOCK: now also R21.2, U1.GP17; no longer U1.GP16
- net N$18: no longer C52.1
- net N$21: now also R23.2, R25.2, T1.C; no longer C64.2
- net N$26: now also L6.1, R26.2; no longer C29.1
- net N$27: now also LED1.A, R18.1; no longer C29.2
- net N$28: now also R22.2, T1.B; no longer C52.2
- net N$7: no longer C64.1
Other:
- moved on the sheet: C16, C17, C18, C19, C20, C21, C22, C29
