File: PCB/Twin_PLL_GPSDO.sch (EAGLE design)
At the start: 136 parts, among them IC1 ADP151WAUJZ-1.8-R7, IC2 ADP151WAUJZ-1.8-R7, IC3 MCP4725A0T-E_CH, IC4 LT1963AEQ-2.5#PBF, T1 BC847, U2 ADF4351BCPZ, U3 ADF4351BCPZ

Commit message: Ketchup
Parts:
- added D1, D2: (no value), diode:DIODE-SOD123
- added R27, R28: 10K, resistor:R-EU_R0603
Connections:
- new net N$40: D1.C, U1.VSYS
- new net N$44: D2.A, R24.1
- net +5V: now also D1.A, R27.2, R28.2; no longer U1.VSYS
- net ALARM_OUT: now also D2.C; no longer R24.1
- net AVDD: now also C38.2, IC3.VDD; no longer C38.1, IC3.VSS
- net GND: now also C38.1, IC3.VSS; no longer C38.2, IC3.VDD
- net I2C_SCL: now also R27.1
- net I2C_SDA: now also R28.1
Changed lines of the file:
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@@
 <part name="R26" library="resistor" deviceset="R-EU_" device="R0603" value="4k7"/>
 <part name="C29" library="rcl" deviceset="C-EU" device="C0805" value="100nF"/>
+<part name="D1" library="diode" deviceset="DIODE-" device="SOD123"/>
+<part name="R27" library="resistor" deviceset="R-EU_" device="R0603" value="10K"/>
+<part name="R28" library="resistor" deviceset="R-EU_" device="R0603" value="10K"/>
+<part name="D2" library="diode" deviceset="DIODE-" device="SOD123"/>
 </parts>
 <sheets>
@@
 <instance part="R26" gate="G$1" x="213.36" y="137.16" rot="R90"/>
 <instance part="C29" gate="G$1" x="378.46" y="284.48"/>
+<instance part="D1" gate="G$1" x="302.26" y="304.8" rot="R180"/>
+<instance part="R27" gate="G$1" x="73.66" y="200.66" rot="R90"/>
+<instance part="R28" gate="G$1" x="78.74" y="190.5" rot="R90"/>
+<instance part="D2" gate="G$1" x="152.4" y="299.72" rot="R180"/>
 </instances>
 <busses>
@@
 <junction x="106.68" y="195.58"/>
 <label x="96.52" y="195.58" size="1.778" layer="95" rot="MR0"/>
-</segment>
-<segment>
-<pinref part="IC3" gate="G$1" pin="VDD"/>
-<wire x1="124.46" y1="170.18" x2="127" y2="170.18" width="0.1524" layer="91"/>
-<label x="137.16" y="160.02" size="1.778" layer="95"/>
-<wire x1="127" y1="170.18" x2="127" y2="160.02" width="0.1524" layer="91"/>
-<pinref part="C38" gate="G$1" pin="2"/>
-<wire x1="127" y1="160.02" x2="132.08" y2="160.02" width="0.1524" layer="91"/>
-<wire x1="132.08" y1="160.02" x2="137.16" y2="160.02" width="0.1524" layer="91"/>
-<junction x="132.08" y="160.02"/>
 </segment>
 <segment>
@@
 <label x="383.54" y="276.86" size="1.778" layer="95"/>
 </segment>
+<segment>
+<pinref part="C38" gate="G$1" pin="1"/>
+<wire x1="132.08" y1="172.72" x2="132.08" y2="167.64" width="0.1524" layer="91"/>
+<pinref part="IC3" gate="G$1" pin="VSS"/>
+<wire x1="124.46" y1="172.72" x2="132.08" y2="172.72" width="0.1524" layer="91"/>
+<wire x1="132.08" y1="172.72" x2="134.62" y2="172.72" width="0.1524" layer="91"/>
+<junction x="132.08" y="172.72"/>
+</segment>
 </net>
 <net name="N$32" class="0">
@@
 <net name="AVDD" class="0">
 <segment>
-<pinref part="IC3" gate="G$1" pin="VSS"/>
-<pinref part="C38" gate="G$1" pin="1"/>
-<wire x1="124.46" y1="172.72" x2="132.08" y2="172.72" width="0.1524" layer="91"/>
-<wire x1="132.08" y1="172.72" x2="132.08" y2="170.18" width="0.1524" layer="91"/>
-<wire x1="132.08" y1="170.18" x2="132.08" y2="167.64" width="0.1524" layer="91"/>
-<junction x="132.08" y="170.18"/>
-<wire x1="132.08" y1="170.18" x2="142.24" y2="170.18" width="0.1524" layer="91"/>
-<wire x1="142.24" y1="170.18" x2="142.24" y2="213.36" width="0.1524" layer="91"/>
+<wire x1="142.24" y1="157.48" x2="142.24" y2="213.36" width="0.1524" layer="91"/>
 <pinref part="C36" gate="G$1" pin="1"/>
 <wire x1="114.3" y1="213.36" x2="114.3" y2="210.82" width="0.1524" layer="91"/>
@@
 <junction x="106.68" y="213.36"/>
 <wire x1="142.24" y1="213.36" x2="114.3" y2="213.36" width="0.1524" layer="91"/>
+<pinref part="IC3" gate="G$1" pin="VDD"/>
+<wire x1="124.46" y1="170.18" x2="127" y2="170.18" width="0.1524" layer="91"/>
+<wire x1="127" y1="170.18" x2="127" y2="157.48" width="0.1524" layer="91"/>
+<pinref part="C38" gate="G$1" pin="2"/>
+<wire x1="127" y1="157.48" x2="132.08" y2="157.48" width="0.1524" layer="91"/>
+<wire x1="132.08" y1="157.48" x2="132.08" y2="160.02" width="0.1524" layer="91"/>
+<wire x1="132.08" y1="157.48" x2="142.24" y2="157.48" width="0.1524" layer="91"/>
+<junction x="132.08" y="157.48"/>
 </segment>
 </net>
@@
 </segment>
 <segment>
-<wire x1="281.94" y1="304.8" x2="289.56" y2="304.8" width="0.1524" layer="91"/>
-<label x="289.56" y="304.8" size="1.778" layer="95" xref="yes"/>
-<pinref part="U1" gate="G$1" pin="VSYS"/>
+<label x="322.58" y="304.8" size="1.778" layer="95" xref="yes"/>
+<pinref part="D1" gate="G$1" pin="A"/>
+<wire x1="304.8" y1="304.8" x2="322.58" y2="304.8" width="0.1524" layer="91"/>
 </segment>
 <segment>
 <pinref part="L8" gate="G$1" pin="2"/>
 <wire x1="86.36" y1="213.36" x2="78.74" y2="213.36" width="0.1524" layer="91"/>
-<label x="78.74" y="213.36" size="1.778" layer="95" rot="MR0" xref="yes"/>
+<label x="55.88" y="213.36" size="1.778" layer="95" rot="MR0" xref="yes"/>
+<pinref part="R27" gate="G$1" pin="2"/>
+<wire x1="78.74" y1="213.36" x2="73.66" y2="213.36" width="0.1524" layer="91"/>
+<wire x1="73.66" y1="213.36" x2="55.88" y2="213.36" width="0.1524" layer="91"/>
+<wire x1="73.66" y1="205.74" x2="73.66" y2="213.36" width="0.1524" layer="91"/>
+<pinref part="R28" gate="G$1" pin="2"/>
+<wire x1="78.74" y1="195.58" x2="78.74" y2="213.36" width="0.1524" layer="91"/>
+<junction x="73.66" y="213.36"/>
+<junction x="78.74" y="213.36"/>
 </segment>
 <segment>
@@
 <segment>
 <pinref part="IC3" gate="G$1" pin="SDA"/>
-<wire x1="96.52" y1="170.18" x2="91.44" y2="170.18" width="0.1524" layer="91"/>
-<label x="91.44" y="170.18" size="1.778" layer="95" rot="R180"/>
+<wire x1="96.52" y1="170.18" x2="78.74" y2="170.18" width="0.1524" layer="91"/>
+<label x="68.58" y="170.18" size="1.778" layer="95" rot="R180"/>
+<wire x1="78.74" y1="170.18" x2="68.58" y2="170.18" width="0.1524" layer="91"/>
+<wire x1="78.74" y1="170.18" x2="78.74" y2="185.42" width="0.1524" layer="91"/>
+<pinref part="R28" gate="G$1" pin="1"/>
+<junction x="78.74" y="170.18"/>
 </segment>
 </net>
@@
 <segment>
 <pinref part="IC3" gate="G$1" pin="SCL"/>
-<wire x1="96.52" y1="172.72" x2="91.44" y2="172.72" width="0.1524" layer="91"/>
-<label x="91.44" y="172.72" size="1.778" layer="95" rot="R180"/>
+<wire x1="96.52" y1="172.72" x2="73.66" y2="172.72" width="0.1524" layer="91"/>
+<label x="68.58" y="172.72" size="1.778" layer="95" rot="R180"/>
+<wire x1="68.58" y1="172.72" x2="73.66" y2="172.72" width="0.1524" layer="91"/>
+<wire x1="73.66" y1="172.72" x2="73.66" y2="195.58" width="0.1524" layer="91"/>
+<pinref part="R27" gate="G$1" pin="1"/>
+<junction x="73.66" y="172.72"/>
 </segment>
 </net>
@@
 <net name="ALARM_OUT" class="0">
 <segment>
-<pinref part="R24" gate="G$1" pin="1"/>
-<wire x1="170.18" y1="299.72" x2="165.1" y2="299.72" width="0.1524" layer="91"/>
-<label x="165.1" y="299.72" size="1.778" layer="95" rot="R180" xref="yes"/>
+<label x="137.16" y="299.72" size="1.778" layer="95" rot="R180" xref="yes"/>
+<wire x1="149.86" y1="299.72" x2="137.16" y2="299.72" width="0.1524" layer="91"/>
+<pinref part="D2" gate="G$1" pin="C"/>
 </segment>
 </net>
@@
 </segment>
 </net>
+<net name="N$40" class="0">
+<segment>
+<pinref part="D1" gate="G$1" pin="C"/>
+<wire x1="281.94" y1="304.8" x2="299.72" y2="304.8" width="0.1524" layer="91"/>
+<pinref part="U1" gate="G$1" pin="VSYS"/>
+</segment>
+</net>
+<net name="N$44" class="0">
+<segment>
+<pinref part="R24" gate="G$1" pin="1"/>
+<pinref part="D2" gate="G$1" pin="A"/>
+<wire x1="170.18" y1="299.72" x2="154.94" y2="299.72" width="0.1524" layer="91"/>
+</segment>
+</net>

Commit message: initial corrections to producion PCB
Parts:
- removed R36, R7: 0R, rcl:R-EU_R0603
- removed R37, R8: NF, rcl:R-EU_R0603
Connections:
- removed net N$15: R5.2, R7.2, R8.1
- removed net N$16: R8.2, U3G$1.SW
- removed net N$49: R34.2, R36.2, R37.1
- removed net N$50: R37.2, U2G$1.SW
- net GND: now also R34.2, R5.2; no longer R36.1, R7.1
Other:
- moved on the sheet: L31
Changed lines of the file:
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@@
 <part name="R35" library="resistor" deviceset="R-EU_" device="R0603" value="680R"/>
 <part name="C56" library="rcl" deviceset="C-EU" device="C0603" value="1N5"/>
-<part name="R36" library="rcl" deviceset="R-EU_" device="R0603" value="0R"/>
-<part name="R37" library="rcl" deviceset="R-EU_" device="R0603" value="NF"/>
 <part name="GND50" library="supply1" deviceset="GND" device=""/>
 <part name="GND51" library="supply1" deviceset="GND" device=""/>
@@
 <part name="R6" library="resistor" deviceset="R-EU_" device="R0603" value="680R"/>
 <part name="C68" library="rcl" deviceset="C-EU" device="C0603" value="1N5"/>
-<part name="R7" library="rcl" deviceset="R-EU_" device="R0603" value="0R"/>
-<part name="R8" library="rcl" deviceset="R-EU_" device="R0603" value="NF"/>
 <part name="GND62" library="supply1" deviceset="GND" device=""/>
 <part name="GND63" library="supply1" deviceset="GND" device=""/>
@@
 <instance part="GND41" gate="1" x="266.7" y="81.28"/>
 <instance part="+3V4" gate="G$1" x="165.1" y="223.52" rot="MR270"/>
-<instance part="+3V5" gate="G$1" x="226.06" y="231.14" rot="MR90"/>
+<instance part="+3V5" gate="G$1" x="226.06" y="233.68" rot="MR90"/>
 <instance part="+3V6" gate="G$1" x="190.5" y="93.98" rot="MR180"/>
 <instance part="+3V7" gate="G$1" x="124.46" y="157.48" rot="MR270"/>
@@
 <instance part="R35" gate="G$1" x="101.6" y="134.62"/>
 <instance part="C56" gate="G$1" x="91.44" y="124.46" rot="R180"/>
-<instance part="R36" gate="G$1" x="106.68" y="162.56"/>
-<instance part="R37" gate="G$1" x="121.92" y="162.56"/>
 <instance part="GND50" gate="1" x="91.44" y="116.84"/>
 <instance part="GND51" gate="1" x="114.3" y="116.84"/>
@@
 <instance part="L32" gate="G$1" x="134.62" y="157.48"/>
 <instance part="L30" gate="G$1" x="175.26" y="223.52"/>
-<instance part="L31" gate="G$1" x="215.9" y="231.14"/>
+<instance part="L31" gate="G$1" x="215.9" y="233.68"/>
 <instance part="L27" gate="G$1" x="248.92" y="127"/>
 <instance part="U$7" gate="CCSA" x="302.26" y="0"/>
@@
 <pinref part="GND41" gate="1" pin="GND"/>
 <pinref part="C51" gate="G$1" pin="1"/>
-</segment>
-<segment>
-<wire x1="101.6" y1="162.56" x2="99.06" y2="162.56" width="0.1524" layer="91"/>
-<pinref part="R36" gate="G$1" pin="1"/>
-<pinref part="GND52" gate="1" pin="GND"/>
 </segment>
 <segment>
@@
 <label x="281.94" y="60.96" size="1.778" layer="95" rot="R180"/>
 </segment>
+<segment>
+<pinref part="GND52" gate="1" pin="GND"/>
+<pinref part="R34" gate="G$1" pin="2"/>
+<wire x1="99.06" y1="162.56" x2="114.3" y2="162.56" width="0.1524" layer="91"/>
+<wire x1="114.3" y1="162.56" x2="114.3" y2="160.02" width="0.1524" layer="91"/>
+</segment>
 </net>
 <net name="+3V3_ADF1" class="0">
@@
 <pinref part="+3V5" gate="G$1" pin="+3V3"/>
 <pinref part="L31" gate="G$1" pin="2"/>
-<wire x1="223.52" y1="231.14" x2="220.98" y2="231.14" width="0.1524" layer="91"/>
+<wire x1="223.52" y1="233.68" x2="220.98" y2="233.68" width="0.1524" layer="91"/>
 </segment>
 </net>
@@
 </segment>
 </net>
-<net name="N$49" class="0">
-<segment>
-<wire x1="114.3" y1="160.02" x2="114.3" y2="162.56" width="0.1524" layer="91"/>
-<wire x1="114.3" y1="162.56" x2="111.76" y2="162.56" width="0.1524" layer="91"/>
-<wire x1="114.3" y1="162.56" x2="116.84" y2="162.56" width="0.1524" layer="91"/>
-<junction x="114.3" y="162.56"/>
-<pinref part="R34" gate="G$1" pin="2"/>
-<pinref part="R36" gate="G$1" pin="2"/>
-<pinref part="R37" gate="G$1" pin="1"/>
-</segment>
-</net>
-<net name="N$50" class="0">
-<segment>
-<wire x1="127" y1="162.56" x2="167.64" y2="162.56" width="0.1524" layer="91"/>
-<pinref part="R37" gate="G$1" pin="2"/>
-<pinref part="U2" gate="G$1" pin="SW"/>
-</segment>
-</net>
 <net name="ADF1_LD" class="0">
 <segment>
@@
 <pinref part="C7" gate="G$1" pin="1"/>
 <pinref part="L31" gate="G$1" pin="1"/>
-<wire x1="210.82" y1="231.14" x2="205.74" y2="231.14" width="0.1524" layer="91"/>
-<wire x1="205.74" y1="231.14" x2="205.74" y2="223.52" width="0.1524" layer="91"/>
+<wire x1="210.82" y1="233.68" x2="205.74" y2="233.68" width="0.1524" layer="91"/>
+<wire x1="205.74" y1="233.68" x2="205.74" y2="223.52" width="0.1524" layer="91"/>
 <junction x="205.74" y="223.52"/>
 </segment>
@@
 <instance part="R6" gate="G$1" x="101.6" y="134.62"/>
 <instance part="C68" gate="G$1" x="91.44" y="124.46" rot="R180"/>
-<instance part="R7" gate="G$1" x="106.68" y="162.56"/>
-<instance part="R8" gate="G$1" x="121.92" y="162.56"/>
 <instance part="GND62" gate="1" x="91.44" y="116.84"/>
 <instance part="GND63" gate="1" x="114.3" y="116.84"/>
@@
 </segment>
 </net>
-<net name="N$15" class="0">
-<segment>
-<wire x1="114.3" y1="160.02" x2="114.3" y2="162.56" width="0.1524" layer="91"/>
-<wire x1="114.3" y1="162.56" x2="111.76" y2="162.56" width="0.1524" layer="91"/>
-<wire x1="114.3" y1="162.56" x2="116.84" y2="162.56" width="0.1524" layer="91"/>
-<junction x="114.3" y="162.56"/>
-<pinref part="R5" gate="G$1" pin="2"/>
-<pinref part="R7" gate="G$1" pin="2"/>
-<pinref part="R8" gate="G$1" pin="1"/>
-</segment>
-</net>
-<net name="N$16" class="0">
-<segment>
-<wire x1="127" y1="162.56" x2="167.64" y2="162.56" width="0.1524" layer="91"/>
-<pinref part="R8" gate="G$1" pin="2"/>
-<pinref part="U3" gate="G$1" pin="SW"/>
-</segment>
-</net>
 <net name="ADF2_LD" class="0">
 <segment>
@@
 <pinref part="GND61" gate="1" pin="GND"/>
 <pinref part="C63" gate="G$1" pin="1"/>
-</segment>
-<segment>
-<wire x1="101.6" y1="162.56" x2="99.06" y2="162.56" width="0.1524" layer="91"/>
-<pinref part="R7" gate="G$1" pin="1"/>
-<pinref part="GND64" gate="1" pin="GND"/>
 </segment>
 <segment>
@@
 <wire x1="274.32" y1="60.96" x2="274.32" y2="71.12" width="0.1524" layer="91"/>
 </segment>
-</net>
+<segment>
+<pinref part="GND64" gate="1" pin="GND"/>
+<pinref part="R5" gate="G$1" pin="2"/>
+<wire x1="99.06" y1="162.56" x2="114.3" y2="162.56" width="0.1524" layer="91"/>
+<wire x1="114.3" y1="162.56" x2="114.3" y2="160.02" width="0.1524" layer="91"/>
+</segment>
+</net>
